Commit message: replace camera with rgbd-kinect

File: urdf/udacity_bot.xacro (robot description, xacro)
@@ -149,5 +149,5 @@
     <inertial>
       <mass value="0.1"/>
-      <origin xyz="0 0 0" rpy="0 0 0"/>
+      <origin xyz="0 0 0" rpy="0 0 1.5708"/>
       <inertia
         ixx="1e-6" ixy="0" ixz="0"
@@ -157,13 +157,13 @@
     </inertial>
     <collision name='camera_collision'>
-      <origin xyz="0 0 0" rpy=" 0 0 0"/>
-      <geometry>
-        <box size="0.05 0.05 0.05" />
+      <origin xyz="0 0 0" rpy=" 0 0 1.5708"/>
+      <geometry>
+        <box size="0.07271 0.27794 0.073" />
       </geometry>
     </collision>
     <visual name='camera_visual'>
-      <origin xyz="0 0 0" rpy=" 0 0 0"/>
-      <geometry>
-        <box size="0.05 0.05 0.05" />
+      <origin xyz="0 0 0" rpy=" 0 0 1.5708"/>
+      <geometry>
+        <mesh filename="package://udacity_bot/meshes/kinect.dae"/>
       </geometry>
     </visual>
@@ -171,5 +171,5 @@
   <!-- camera + chassis JOINT -->
   <joint type="fixed" name="camera_joint">
-    <origin xyz="0.2 0 0" rpy="0 0 0"/>
+    <origin xyz="0.25 0 0" rpy="0 0 0"/>
     <child link="camera"/>
     <parent link="chassis"/>

Commit message: rename camera to kinect

File: urdf/udacity_bot.xacro (robot description, xacro)
@@ -145,6 +145,6 @@
     <joint_properties damping="1.0" friction="1.0"/>
   </joint>
-  <!-- camera - LINK -->
-  <link name='camera'>
+  <!-- kinect - LINK -->
+  <link name='kinect'>
     <inertial>
       <mass value="0.1"/>
@@ -156,5 +156,5 @@
       />
     </inertial>
-    <collision name='camera_collision'>
+    <collision name='kinect_collision'>
       <origin xyz="0 0 0" rpy=" 0 0 1.5708"/>
       <geometry>
@@ -162,5 +162,5 @@
       </geometry>
     </collision>
-    <visual name='camera_visual'>
+    <visual name='kinect_visual'>
       <origin xyz="0 0 0" rpy=" 0 0 1.5708"/>
       <geometry>
@@ -169,8 +169,8 @@
     </visual>
   </link>
-  <!-- camera + chassis JOINT -->
-  <joint type="fixed" name="camera_joint">
+  <!-- kinect + chassis JOINT -->
+  <joint type="fixed" name="kinect_joint">
     <origin xyz="0.25 0 0" rpy="0 0 0"/>
-    <child link="camera"/>
+    <child link="kinect"/>
     <parent link="chassis"/>
   </joint>

Commit message: solve point cloud on z-axis

File: urdf/udacity_bot.xacro (robot description, xacro)
@@ -149,5 +149,5 @@
     <inertial>
       <mass value="0.1"/>
-      <origin xyz="0 0 0" rpy="0 0 1.5708"/>
+      <origin xyz="0 0 0" rpy="0 0 0"/>
       <inertia
         ixx="1e-6" ixy="0" ixz="0"
@@ -157,5 +157,5 @@
     </inertial>
     <collision name='kinect_collision'>
-      <origin xyz="0 0 0" rpy=" 0 0 1.5708"/>
+      <origin xyz="0 0 0" rpy="0 0 0"/>
       <geometry>
         <box size="0.07271 0.27794 0.073" />
@@ -163,5 +163,5 @@
     </collision>
     <visual name='kinect_visual'>
-      <origin xyz="0 0 0" rpy=" 0 0 1.5708"/>
+      <origin xyz="0 0 0" rpy="0 0 1.5708"/>
       <geometry>
         <mesh filename="package://udacity_bot/meshes/kinect.dae"/>

Commit message: UPDATE: xarco

File: urdf/udacity_bot.xacro (robot description, xacro)
@@ -149,5 +149,4 @@
     <inertial>
       <mass value="0.1"/>
-      <origin xyz="0 0 0" rpy="0 0 1.5708"/>
       <inertia
         ixx="1e-6" ixy="0" ixz="0"
@@ -157,5 +156,4 @@
     </inertial>
     <collision name='kinect_collision'>
-      <origin xyz="0 0 0" rpy=" 0 0 1.5708"/>
       <geometry>
         <box size="0.07271 0.27794 0.073" />
@@ -163,5 +161,4 @@
     </collision>
     <visual name='kinect_visual'>
-      <origin xyz="0 0 0" rpy=" 0 0 1.5708"/>
       <geometry>
         <mesh filename="package://udacity_bot/meshes/kinect.dae"/>
@@ -171,5 +168,5 @@
   <!-- kinect + chassis JOINT -->
   <joint type="fixed" name="kinect_joint">
-    <origin xyz="0.25 0 0" rpy="0 0 0"/>
+    <origin xyz="0.25 0 0" rpy="0 0 1.5708"/>
     <child link="kinect"/>
     <parent link="chassis"/>

Commit message: Replace base from robot_foot to chassis

File: urdf/udacity_bot.xacro (robot description, xacro)
@@ -2,12 +2,4 @@
 <robot name="udacity_bot" xmlns:xacro="http://www.ros.org/wiki/xacro">
   <xacro:include filename="$(find udacity_bot)/urdf/udacity_bot.gazebo" />
-  <!-- footprint LINK -->
-  <link name="robot_footprint"></link>
-  <!-- footprint + chassis JOINT -->
-  <joint name="robot_footprint_joint" type="fixed">
-    <origin xyz="0 0 0" rpy="0 0 0" />
-    <parent link="robot_footprint"/>
-    <child link="chassis" />
-  </joint>
   <!-- chassis LINK -->
   <link name='chassis'>
