Commit message: update urdf

File: urdf/slam.xacro (robot description, xacro)
@@ -5,4 +5,5 @@
   <xacro:include filename="$(find udacity_bot)/urdf/slam/right_wheel.xacro" />
   <xacro:include filename="$(find udacity_bot)/urdf/slam/left_wheel.xacro" />
+  <xacro:include filename="$(find udacity_bot)/urdf/slam/rod.xacro" />
   <xacro:include filename="$(find udacity_bot)/urdf/slam/kinect.xacro" />
   <xacro:include filename="$(find udacity_bot)/urdf/slam/laser.xacro" />

File: urdf/slam/kinect.xacro (robot description, xacro)
@@ -27,7 +27,7 @@
   <!-- kinect + chassis JOINT -->
   <joint type="fixed" name="kinect_joint">
-    <origin xyz="0.25 0 0" rpy="0 0 0"/>
+    <origin xyz="0 0 0.2" rpy="0 0 0"/>
     <child link="kinect"/>
-    <parent link="chassis"/>
+    <parent link="rod"/>
   </joint>
 </robot>
